File: BoardGame.kicad_pcb (KiCad board)
At the start: 2 copper layers, 32 parts, among them J1 Conn_01x10_Male, Q1 VP3203N3-G, Q2 VP3203N3-G, Q3 VP3203N3-G, SW1 SW_Push_11_22, SW2 SW_Push_11_22, SW3 SW_Push_11_22, SW4 SW_Push_11_22, SW5 SW_Push_11_22, SW6 SW_Push_11_22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

Commit message: Added caps to PCB
I added cap footprints to the PCB
Parts:
- added C1: 1uF, Capacitor_THT:CP_Radial_D5.0mm_P2.50mm, F.Cu at (135.1, 101.2)
- added C2: 0.1uF, Capacitor_THT:C_Rect_L4.6mm_W3.0mm_P2.50mm_MKS02_FKP02, F.Cu at (77.1, 100.2)
- added C3: 0.1uF, Capacitor_THT:C_Rect_L4.6mm_W3.0mm_P2.50mm_MKS02_FKP02, F.Cu at (125.1, 100.2)
- added C4: 0.1uF, Capacitor_THT:C_Rect_L4.6mm_W3.0mm_P2.50mm_MKS02_FKP02, F.Cu at (101.1, 100.2)
- added C5: 0.1uF, Capacitor_THT:C_Rect_L4.6mm_W3.0mm_P2.50mm_MKS02_FKP02, F.Cu at (33.1, 50.2)
