File: BoardGame.sch (KiCad schematic (older format))
At the start: 20 parts, among them J1 Conn_01x10_Male, SW1 SW_Push_11_22, SW2 SW_Push_11_22, SW3 SW_Push_11_22, SW4 SW_Push_11_22, SW5 SW_Push_11_22, SW6 SW_Push_11_22, SW7 SW_Push_11_22, SW8 SW_Push_11_22, SW9 SW_Push_11_22

Commit message: Added caps to PCB
I added cap footprints to the PCB
Parts:
- C1: footprint (none) -> Capacitor_THT:CP_Radial_D5.0mm_P2.50mm
Changed lines of the file:
@@
 F 0 "C1" H 10965 1846 50  0000 L CNN
 F 1 "1uF" H 10965 1755 50  0000 L CNN
-F 2 "" H 10888 1650 50  0001 C CNN
+F 2 "Capacitor_THT:CP_Radial_D5.0mm_P2.50mm" H 10888 1650 50  0001 C CNN
 F 3 "~" H 10850 1800 50  0001 C CNN
 	1    10850 1800
