File: ColumnDriverP.sch (KiCad schematic (older format))
At the start: 5 parts, among them Q1 VP3203N3-G, Q2 VP3203N3-G, Q3 VP3203N3-G, U4 74HCT595

Commit message: Added caps to PCB
I added cap footprints to the PCB
Parts:
- C5: footprint (none) -> Capacitor_THT:C_Rect_L4.6mm_W3.0mm_P2.50mm_MKS02_FKP02
Changed lines of the file:
@@
 F 0 "C5" H 4015 1596 50  0000 L CNN
 F 1 "0.1uF" H 4015 1505 50  0000 L CNN
-F 2 "" H 3938 1400 50  0001 C CNN
+F 2 "Capacitor_THT:C_Rect_L4.6mm_W3.0mm_P2.50mm_MKS02_FKP02" H 3938 1400 50  0001 C CNN
 F 3 "~" H 3900 1550 50  0001 C CNN
 	1    3900 1550
