File: RowDriverN.sch (KiCad schematic (older format))
At the start: 12 parts, among them U1 TLC5916, U2 TLC5916, U3 74HCT165

Commit message: Added caps to PCB
I added cap footprints to the PCB
Parts:
- C2, C3, C4: footprint (none) -> Capacitor_THT:C_Rect_L4.6mm_W3.0mm_P2.50mm_MKS02_FKP02
Changed lines of the file:
@@
 F 0 "C4" H 6315 1896 50  0000 L CNN
 F 1 "0.1uF" H 6315 1805 50  0000 L CNN
-F 2 "" H 6238 1700 50  0001 C CNN
+F 2 "Capacitor_THT:C_Rect_L4.6mm_W3.0mm_P2.50mm_MKS02_FKP02" H 6238 1700 50  0001 C CNN
 F 3 "~" H 6200 1850 50  0001 C CNN
 	1    6200 1850
@@
 F 0 "C3" H 3715 5396 50  0000 L CNN
 F 1 "0.1uF" H 3715 5305 50  0000 L CNN
-F 2 "" H 3638 5200 50  0001 C CNN
+F 2 "Capacitor_THT:C_Rect_L4.6mm_W3.0mm_P2.50mm_MKS02_FKP02" H 3638 5200 50  0001 C CNN
 F 3 "~" H 3600 5350 50  0001 C CNN
 	1    3600 5350
@@
 F 0 "C2" H 3715 3546 50  0000 L CNN
 F 1 "0.1uF" H 3715 3455 50  0000 L CNN
-F 2 "" H 3638 3350 50  0001 C CNN
+F 2 "Capacitor_THT:C_Rect_L4.6mm_W3.0mm_P2.50mm_MKS02_FKP02" H 3638 3350 50  0001 C CNN
 F 3 "~" H 3600 3500 50  0001 C CNN
 	1    3600 3500

Commit message: Update RowDriverN.sch
Cleaned up row driver parts to point to correct datasheet.
changed resistors to 1k for switches and level shifts and rext where they program about 20ma of LED current.
Parts:
- R1, R2: value R_US -> 1k
- R3, R4, R5, R6: value 10k -> 1k
Other:
- moved on the sheet: U2
Changed lines of the file:
@@
 U 1 1 5DE85293
 P 5850 2800
-F 0 "U3" H 5850 3581 50  0000 C CNN
-F 1 "74HCT165" H 5850 3490 50  0000 C CNN
+F 0 "U3" H 5600 3450 50  0000 C CNN
+F 1 "74HCT165" H 5550 3350 50  0000 C CNN
 F 2 "Package_DIP:DIP-16_W7.62mm" H 5850 2800 50  0001 C CNN
 F 3 "https://assets.nexperia.com/documents/data-sheet/74HC_HCT165.pdf" H 5850 2800 50  0001 C CNN
@@
 Text HLabel 4050 4450 2    50   Output ~ 0
 GLEDR2
-Text HLabel 4050 5900 2    50   Output ~ 0
+Text HLabel 4250 5900 2    50   Output ~ 0
 BLEDR2
-Text HLabel 4050 6000 2    50   Output ~ 0
+Text HLabel 4250 6000 2    50   Output ~ 0
 RLEDR3
-Text HLabel 4050 6100 2    50   Output ~ 0
+Text HLabel 4250 6100 2    50   Output ~ 0
 GLEDR3
-Text HLabel 4050 6200 2    50   Output ~ 0
+Text HLabel 4250 6200 2    50   Output ~ 0
 BLEDR3
 Text HLabel 5000 3550 0    50   Output ~ 0
@@
 P 6350 3850
 F 0 "R4" H 6418 3896 50  0000 L CNN
-F 1 "10k" H 6418 3805 50  0000 L CNN
+F 1 "1k" H 6418 3805 50  0000 L CNN
 F 2 "Resistor_THT:R_Axial_DIN0207_L6.3mm_D2.5mm_P7.62mm_Horizontal" V 6390 3840 50  0001 C CNN
 F 3 "~" H 6350 3850 50  0001 C CNN
@@
 P 6650 3700
 F 0 "R5" H 6718 3746 50  0000 L CNN
-F 1 "10k" H 6718 3655 50  0000 L CNN
+F 1 "1k" H 6718 3655 50  0000 L CNN
 F 2 "Resistor_THT:R_Axial_DIN0207_L6.3mm_D2.5mm_P7.62mm_Horizontal" V 6690 3690 50  0001 C CNN
 F 3 "~" H 6650 3700 50  0001 C CNN
@@
 P 6950 3850
 F 0 "R6" H 7018 3896 50  0000 L CNN
-F 1 "10k" H 7018 3805 50  0000 L CNN
+F 1 "1k" H 7018 3805 50  0000 L CNN
 F 2 "Resistor_THT:R_Axial_DIN0207_L6.3mm_D2.5mm_P7.62mm_Horizontal" V 6990 3840 50  0001 C CNN
 F 3 "~" H 6950 3850 50  0001 C CNN
@@
 U 1 1 5DDE8EE0
 P 3250 4750
-F 0 "U1" H 3250 5931 50  0000 C CNN
-F 1 "TLC5916" H 3250 5840 50  0000 C CNN
+F 0 "U1" H 2800 5700 50  0000 C CNN
+F 1 "TLC5916" H 2900 5600 50  0000 C CNN
 F 2 "Package_DIP:DIP-16_W7.62mm" H 3300 3775 50  0001 L CNN
-F 3 "http://www.ti.com/lit/ds/symlink/tlc5940.pdf" H 2850 5450 50  0001 C CNN
+F 3 "http://www.ti.com/lit/ds/symlink/tlc5916.pdf" H 2850 5450 50  0001 C CNN
 	1    3250 4750
 	1    0    0    -1
@@
 P 5200 3550
 F 0 "R3" H 5268 3596 50  0000 L CNN
-F 1 "10k" H 5268 3505 50  0000 L CNN
+F 1 "1k" H 5268 3505 50  0000 L CNN
 F 2 "Resistor_THT:R_Axial_DIN0207_L6.3mm_D2.5mm_P7.62mm_Horizontal" V 5240 3540 50  0001 C CNN
 F 3 "~" H 5200 3550 50  0001 C CNN
@@
 L tlc5916:TLC5916 U2
 U 1 1 5E184EC9
-P 3250 6600
-F 0 "U2" H 3250 7781 50  0000 C CNN
-F 1 "TLC5916" H 3250 7690 50  0000 C CNN
-F 2 "Package_DIP:DIP-16_W7.62mm" H 3300 5625 50  0001 L CNN
-F 3 "http://www.ti.com/lit/ds/symlink/tlc5940.pdf" H 2850 7300 50  0001 C CNN
-	1    3250 6600
+P 3450 6600
+F 0 "U2" H 3000 7550 50  0000 C CNN
+F 1 "TLC5916" H 3100 7450 50  0000 C CNN
+F 2 "Package_DIP:DIP-16_W7.62mm" H 3500 5625 50  0001 L CNN
+F 3 "http://www.ti.com/lit/ds/symlink/tlc5916.pdf" H 3050 7300 50  0001 C CNN
+	1    3450 6600
 	1    0    0    -1
 $EndComp
@@
 L power:GND #PWR08
 U 1 1 5E1867D7
-P 3250 6950
-F 0 "#PWR08" H 3250 6700 50  0001 C CNN
-F 1 "GND" H 3255 6777 50  0000 C CNN
-F 2 "" H 3250 6950 50  0001 C CNN
-F 3 "" H 3250 6950 50  0001 C CNN
-	1    3250 6950
+P 3450 6950
+F 0 "#PWR08" H 3450 6700 50  0001 C CNN
+F 1 "GND" H 3455 6777 50  0000 C CNN
+F 2 "" H 3450 6950 50  0001 C CNN
+F 3 "" H 3450 6950 50  0001 C CNN
+	1    3450 6950
 	1    0    0    -1
 $EndComp
@@
 	3250 5050 3250 5100
 Wire Wire Line
-	3250 6900 3250 6950
+	3450 6900 3450 6950
 Wire Wire Line
 	2550 4750 2500 4750
@@
 	2500 4750 2500 6500
 Wire Wire Line
-	2500 6500 2550 6500
-Wire Wire Line
-	2550 6400 2450 6400
-Wire Wire Line
 	2450 4550 2550 4550
 Wire Wire Line
@@
 	3950 4450 4050 4450
 Wire Wire Line
-	4050 5900 3950 5900
-Wire Wire Line
-	3950 6000 4050 6000
-Wire Wire Line
-	4050 6100 3950 6100
-Wire Wire Line
-	3950 6200 4050 6200
+	4250 5900 4150 5900
+Wire Wire Line
+	4150 6000 4250 6000
+Wire Wire Line
+	4250 6100 4150 6100
+Wire Wire Line
+	4150 6200 4250 6200
 Wire Wire Line
 	2550 4250 2400 4250
 Wire Wire Line
 	2400 4250 2400 6100
-Wire Wire Line
-	2400 6100 2550 6100
 $Comp
 L Device:R_US R1
@@
 P 2050 4850
 F 0 "R1" H 2118 4896 50  0000 L CNN
-F 1 "R_US" H 2118 4805 50  0000 L CNN
+F 1 "1k" H 2118 4805 50  0000 L CNN
 F 2 "Resistor_THT:R_Axial_DIN0207_L6.3mm_D2.5mm_P7.62mm_Horizontal" V 2090 4840 50  0001 C CNN
 F 3 "~" H 2050 4850 50  0001 C CNN
@@
 P 2100 6400
 F 0 "R2" H 2168 6446 50  0000 L CNN
-F 1 "R_US" H 2168 6355 50  0000 L CNN
+F 1 "1k" H 2168 6355 50  0000 L CNN
 F 2 "Resistor_THT:R_Axial_DIN0207_L6.3mm_D2.5mm_P7.62mm_Horizontal" V 2140 6390 50  0001 C CNN
 F 3 "~" H 2100 6400 50  0001 C CNN
@@
 	1    0    0    -1
 $EndComp
-Wire Wire Line
-	2550 6000 2100 6000
 Wire Wire Line
 	2100 6000 2100 6250
@@
 	2350 4350 2350 6200
 Wire Wire Line
-	2350 6200 2550 6200
-Wire Wire Line
 	2350 4350 2550 4350
 Connection ~ 2400 4250
@@
 $EndComp
 Wire Wire Line
-	5850 2200 6050 2200
-Wire Wire Line
-	6050 2200 6050 1650
-Wire Wire Line
-	6050 1650 6200 1650
+	5850 2200 5850 1650
+Wire Wire Line
+	5850 1650 6200 1650
 Wire Wire Line
 	6200 1650 6200 1600
@@
 $EndComp
 Wire Wire Line
-	3250 5600 3450 5600
-Wire Wire Line
 	3450 5600 3450 5150
 Wire Wire Line
@@
 $EndComp
 Wire Wire Line
-	3250 3750 3450 3750
-Wire Wire Line
-	3450 3750 3450 3300
-Wire Wire Line
-	3450 3300 3600 3300
+	3250 3750 3250 3300
+Wire Wire Line
+	3250 3300 3600 3300
 Wire Wire Line
 	3600 3300 3600 3350
@@
 NoConn ~ 3950 4650
 NoConn ~ 3950 4750
-NoConn ~ 3950 6300
-NoConn ~ 3950 6400
-NoConn ~ 3950 6500
-NoConn ~ 3950 6600
+NoConn ~ 4150 6300
+NoConn ~ 4150 6400
+NoConn ~ 4150 6500
+NoConn ~ 4150 6600
 Wire Wire Line
 	5450 2400 5000 2400
@@
 	6450 3100 6450 3150
 Connection ~ 6450 3100
-NoConn ~ 2550 6600
+NoConn ~ 2750 6600
+Wire Wire Line
+	2500 6500 2750 6500
+Wire Wire Line
+	2450 6400 2750 6400
+Wire Wire Line
+	2350 6200 2750 6200
+Wire Wire Line
+	2400 6100 2750 6100
+Wire Wire Line
+	2100 6000 2750 6000
 $EndSCHEMATC
